File: Matrix.kicad_sch (KiCad schematic)
At the start: 134 parts, among them SW1 SW_Push, SW10 SW_Push, SW11 SW_Push, SW12 SW_Push, SW13 SW_Push, SW14 SW_Push, SW15 SW_Push, SW16 SW_Push, SW17 SW_Push, SW18 SW_Push, SW19 SW_Push, SW2 SW_Push, SW20 SW_Push, SW21 SW_Push, SW22 SW_Push, SW23 SW_Push, SW24 SW_Push, SW25 SW_Push, SW26 SW_Push, SW27 SW_Push, SW28 SW_Push, SW29 SW_Push, SW3 SW_Push, SW30 SW_Push, SW31 SW_Push, SW32 SW_Push, SW33 SW_Push, SW34 SW_Push, SW35 SW_Push, SW36 SW_Push, SW37 SW_Push, SW38 SW_Push, SW39 SW_Push, SW4 SW_Push, SW40 SW_Push, SW41 SW_Push, SW42 SW_Push, SW43 SW_Push, SW44 SW_Push, SW45 SW_Push, SW46 SW_Push, SW47 SW_Push, SW48 SW_Push, SW49 SW_Push, SW5 SW_Push, SW50 SW_Push, SW51 SW_Push, SW52 SW_Push, SW53 SW_Push, SW54 SW_Push, SW55 SW_Push, SW56 SW_Push, SW57 SW_Push, SW58 SW_Push, SW59 SW_Push, SW6 SW_Push, SW60 SW_Push, SW61 SW_Push, SW62 SW_Push, SW63 SW_Push, SW64 SW_Push, SW65 SW_Push, SW66 SW_Push, SW67 SW_Push, SW7 SW_Push, SW8 SW_Push, SW9 SW_Push

Commit message: Schema finished
Parts:
- D1, D10, D11, D12, D13, D14, D15, D16, D17, D18, D19, D2, D20, D21, D22, D23, D24, D25, D26, D27, D28, D29, D3, D30, D31, D32, D33, D34, D35, D36, D37, D38, D39, D4, D40, D41, D42, D43, D44, D45, D46, D47, D48, D49, D5, D50, D51, D52, D53, D54, D55, D56, D57, D58, D59, D6, D60, D61, D62, D63, D64, D65, D66, D67, D7, D8, D9: footprint (none) -> Diode_SMD:D_SOD-123
- SW1: value SW_Push -> GRV; footprint (none) -> MX_Alps_Hybrid:MX-1U-NoLED
- SW10: value SW_Push -> #9; footprint (none) -> MX_Alps_Hybrid:MX-1U-NoLED
- SW11: value SW_Push -> #0; footprint (none) -> MX_Alps_Hybrid:MX-1U-NoLED
- SW12: value SW_Push -> -_; footprint (none) -> MX_Alps_Hybrid:MX-1U-NoLED
- SW13: value SW_Push -> =+; footprint (none) -> MX_Alps_Hybrid:MX-1U-NoLED
- SW14: value SW_Push -> BSPC; footprint (none) -> MX_Alps_Hybrid:MX-2U-NoLED
- SW15: value SW_Push -> PGUP; footprint (none) -> MX_Alps_Hybrid:MX-1U-NoLED
- SW16: value SW_Push -> TAB; footprint (none) -> MX_Alps_Hybrid:MX-1.5U-NoLED
- SW17: value SW_Push -> Q; footprint (none) -> MX_Alps_Hybrid:MX-1U-NoLED
- SW18: value SW_Push -> W; footprint (none) -> MX_Alps_Hybrid:MX-1U-NoLED
- SW19: value SW_Push -> E; footprint (none) -> MX_Alps_Hybrid:MX-1U-NoLED
- SW2: value SW_Push -> #1; footprint (none) -> MX_Alps_Hybrid:MX-1U-NoLED
- SW20: value SW_Push -> R; footprint (none) -> MX_Alps_Hybrid:MX-1U-NoLED
- SW21: value SW_Push -> T; footprint (none) -> MX_Alps_Hybrid:MX-1U-NoLED
- SW22: value SW_Push -> Y; footprint (none) -> MX_Alps_Hybrid:MX-1U-NoLED
- SW23: value SW_Push -> U; footprint (none) -> MX_Alps_Hybrid:MX-1U-NoLED
- SW24: value SW_Push -> I; footprint (none) -> MX_Alps_Hybrid:MX-1U-NoLED
- SW25: value SW_Push -> O; footprint (none) -> MX_Alps_Hybrid:MX-1U-NoLED
- SW26: value SW_Push -> P; footprint (none) -> MX_Alps_Hybrid:MX-1U-NoLED
- SW27: value SW_Push -> [{; footprint (none) -> MX_Alps_Hybrid:MX-1U-NoLED
- SW28: value SW_Push -> ]}; footprint (none) -> MX_Alps_Hybrid:MX-1U-NoLED
- SW29: value SW_Push -> \|; footprint (none) -> MX_Alps_Hybrid:MX-1.5U-NoLED
- SW3: value SW_Push -> #2; footprint (none) -> MX_Alps_Hybrid:MX-1U-NoLED
- SW30: value SW_Push -> PGDN; footprint (none) -> MX_Alps_Hybrid:MX-1U-NoLED
- SW31: value SW_Push -> CPLK; footprint (none) -> MX_Alps_Hybrid:MX-1.75U-NoLED
- SW32: value SW_Push -> A; footprint (none) -> MX_Alps_Hybrid:MX-1U-NoLED
- SW33: value SW_Push -> S; footprint (none) -> MX_Alps_Hybrid:MX-1U-NoLED
- SW34: value SW_Push -> D; footprint (none) -> MX_Alps_Hybrid:MX-1U-NoLED
- SW35: value SW_Push -> F; footprint (none) -> MX_Alps_Hybrid:MX-1U-NoLED
- SW36: value SW_Push -> G; footprint (none) -> MX_Alps_Hybrid:MX-1U-NoLED
- SW37: value SW_Push -> H; footprint (none) -> MX_Alps_Hybrid:MX-1U-NoLED
- SW38: value SW_Push -> J; footprint (none) -> MX_Alps_Hybrid:MX-1U-NoLED
- SW39: value SW_Push -> K; footprint (none) -> MX_Alps_Hybrid:MX-1U-NoLED
- SW4: value SW_Push -> #3; footprint (none) -> MX_Alps_Hybrid:MX-1U-NoLED
- SW40: value SW_Push -> L; footprint (none) -> MX_Alps_Hybrid:MX-1U-NoLED
- SW41: value SW_Push -> ;:; footprint (none) -> MX_Alps_Hybrid:MX-1U-NoLED
- SW42: value SW_Push -> '"; footprint (none) -> MX_Alps_Hybrid:MX-1U-NoLED
- SW43: value SW_Push -> ENTR; footprint (none) -> MX_Alps_Hybrid:MX-2.25U-NoLED
- SW44: value SW_Push -> INSR; footprint (none) -> MX_Alps_Hybrid:MX-1U-NoLED
- SW45: value SW_Push -> SHFT; footprint (none) -> MX_Alps_Hybrid:MX-2.25U-NoLED
- SW46: value SW_Push -> Z; footprint (none) -> MX_Alps_Hybrid:MX-1U-NoLED
- SW47: value SW_Push -> X; footprint (none) -> MX_Alps_Hybrid:MX-1U-NoLED
- SW48: value SW_Push -> C; footprint (none) -> MX_Alps_Hybrid:MX-1U-NoLED
- SW49: value SW_Push -> V; footprint (none) -> MX_Alps_Hybrid:MX-1U-NoLED
- SW5: value SW_Push -> #4; footprint (none) -> MX_Alps_Hybrid:MX-1U-NoLED
- SW50: value SW_Push -> B; footprint (none) -> MX_Alps_Hybrid:MX-1U-NoLED
- SW51: value SW_Push -> N; footprint (none) -> MX_Alps_Hybrid:MX-1U-NoLED
- SW52: value SW_Push -> M; footprint (none) -> MX_Alps_Hybrid:MX-1U-NoLED
- SW53: value SW_Push -> ,<; footprint (none) -> MX_Alps_Hybrid:MX-1U-NoLED
- SW54: value SW_Push -> .>; footprint (none) -> MX_Alps_Hybrid:MX-1U-NoLED
- SW55: value SW_Push -> /?; footprint (none) -> MX_Alps_Hybrid:MX-1U-NoLED
- SW56: value SW_Push -> SHFT; footprint (none) -> MX_Alps_Hybrid:MX-1.75U-NoLED
- SW57: value SW_Push -> UP; footprint (none) -> MX_Alps_Hybrid:MX-1U-NoLED
- SW58: value SW_Push -> DELT; footprint (none) -> MX_Alps_Hybrid:MX-1U-NoLED
- SW59: value SW_Push -> CTRL; footprint (none) -> MX_Alps_Hybrid:MX-1.5U-NoLED
- SW6: value SW_Push -> #5; footprint (none) -> MX_Alps_Hybrid:MX-1U-NoLED
- SW60, SW63: value SW_Push -> ALT; footprint (none) -> MX_Alps_Hybrid:MX-1.25U-NoLED
- SW61: value SW_Push -> COMD; footprint (none) -> MX_Alps_Hybrid:MX-1.5U-NoLED
- SW62: value SW_Push -> SPAC; footprint (none) -> MX_Alps_Hybrid:MX-6.5U-NoLED
- SW64: value SW_Push -> 0; footprint (none) -> MX_Alps_Hybrid:MX-1U-NoLED
- SW65: value SW_Push -> LEFT; footprint (none) -> MX_Alps_Hybrid:MX-1U-NoLED
- SW66: value SW_Push -> DOWN; footprint (none) -> MX_Alps_Hybrid:MX-1U-NoLED
- SW67: value SW_Push -> RGHT; footprint (none) -> MX_Alps_Hybrid:MX-1U-NoLED
- SW7: value SW_Push -> #6; footprint (none) -> MX_Alps_Hybrid:MX-1U-NoLED
- SW8: value SW_Push -> #7; footprint (none) -> MX_Alps_Hybrid:MX-1U-NoLED
- SW9: value SW_Push -> #8; footprint (none) -> MX_Alps_Hybrid:MX-1U-NoLED
