File: keyboard-design-practice.kicad_pcb (KiCad board)
At the start: 2 copper layers, 155 parts, among them J1 AVR-ISP-6, SW1 GRV, SW10 #9, SW11 #0, SW12 -_, SW13 =+, SW14 BSPC, SW15 PGUP, SW16 TAB, SW17 Q, SW18 W, SW19 E, SW2 #1, SW20 R, SW21 T, SW22 Y, SW23 U, SW24 I, SW25 O, SW26 P, SW27 [{, SW28 ]}, SW29 \|, SW3 #2, SW30 PGDN, SW31 CPLK, SW32 A, SW33 S, SW34 D, SW35 F, SW36 G, SW37 H, SW38 J, SW39 K, SW4 #3, SW40 L, SW41 ;:, SW42 '", SW43 ENTR, SW44 INSR, SW45 SHFT, SW46 Z, SW47 X, SW48 C, SW49 V, SW5 #4, SW50 B, SW51 N, SW52 M, SW53 ,<, SW54 .>, SW55 /?, SW56 SHFT, SW57 UP, SW58 DELT, SW59 CTRL, SW6 #5, SW60 ALT, SW61 COMD, SW62 SPAC, SW63 ALT, SW64 0, SW65 LEFT, SW66 DOWN, SW67 RGHT, SW68 SW_Push, SW7 #6, SW8 #7, SW9 #8, U1 ATmega32U4-A, U2 PRTR5V0U2X, Y1 16MHz

Commit message: All footprints in place
Parts:
- moved USB1 172.8 mm to (191.3, 64.5), turned to 0 degrees
- moved R5 161.7 mm to (193.7, 77.0), turned to 0 degrees
- moved F1 161.4 mm to (187.3, 84.9), turned to -90 degrees
- moved R6 159.3 mm to (188.9, 77.0)
- moved U2 156.8 mm to (191.3, 83.3), turned to 0 degrees
- moved R3 114.5 mm to (208.8, 140.5), turned to -90 degrees
- moved R4 113.9 mm to (211.1, 140.5), turned to 90 degrees
- moved SW68 109.8 mm to (239.4, 153.1), turned to 90 degrees
- moved C7 109.7 mm to (225.4, 155.6), turned to 0 degrees
- moved C2 109.7 mm to (215.9, 149.2), turned to 90 degrees
- moved C6 107.0 mm to (225.4, 153.2), turned to 0 degrees
- moved C5 106.2 mm to (211.1, 145.3)
- moved C4 103.0 mm to (200.0, 146.1)
- moved C8 101.3 mm to (207.2, 145.3)
- moved Y1 99.7 mm to (219.7, 154.3), turned to 0 degrees
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Other:
- board outline added: 304.8 x 99.2 mm

Commit message: little changes
Parts:
- moved R1 48.4 mm to (217.5, 115.9)
- moved C4 39.5 mm to (184.9, 109.5)
- moved SW20 39.5 mm to (119.1, 61.9)
- moved SW22 39.5 mm to (157.2, 61.9)
- moved SW24 39.5 mm to (195.3, 61.9)
- moved SW25 39.5 mm to (214.3, 61.9)
- moved SW28 39.5 mm to (271.5, 61.9)
- moved SW29 39.5 mm to (295.3, 61.9)
- moved SW30 39.5 mm to (319.1, 61.9)
- moved D1 39.5 mm to (29.4, 46.8)
- moved D10 39.5 mm to (200.8, 46.8)
- moved D12 39.5 mm to (238.9, 46.8)
- moved D13 39.5 mm to (258.0, 46.8)
- moved D14 39.5 mm to (286.5, 46.8)
- moved D15 39.5 mm to (315.1, 46.8)
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